File: eagle/control project.sch (EAGLE design)
At the start: 29 parts, among them IC1 7805TV, IC3 MEGA32-P, Q1 16Mhz

Commit message: v4
Parts:
- added ANALONG: (no value), pinhead:PINHD-1X4
- added C2: 10uf, rcl:C-EU102-043X133
- added R5, R7, R8: (no value), rcl:POTENTIOMETER_PT-10
- added R6, R9: 10k, rcl:R-EU_0204/7
- added S2, S3: (no value), switch-omron:10-XX
- added SEND: (no value), pinhead:PINHD-1X3
Connections:
- removed net N$12: IC3.(ADC2)PA2, JP1.6
- removed net N$13: IC3.(ADC1)PA1, JP1.7
- removed net N$14: IC3.(ADC0)PA0, JP1.8
- removed net N$41: IC3.(INT0)PD2, JP2.6
- removed net N$42: IC3.(TXD)PD1, JP2.7
- removed net N$43: IC3.(RXD)PD0, JP2.8
- new net A0: IC3.(ADC0)PA0, JP1.8, R8.3
- new net A1: IC3.(ADC1)PA1, JP1.7, R7.3
- new net A2: IC3.(ADC2)PA2, JP1.6, R5.3
- new net AREF: ANALONG.1, C2.2, IC3.AREF
- new net AVCC: ANALONG.2, IC3.AVCC
- new net IN0: IC3.(INT0)PD2, JP2.6, R9.1, S3.S, S3.S1
- new net IN1: IC3.(INT1)PD3, JP2.5, L298N.5, R6.1, S2.S, S2.S1
- new net RX: IC3.(RXD)PD0, JP2.8, SEND.2
- new net TX: IC3.(TXD)PD1, JP2.7, SEND.1
- net +5V: now also ANALONG.3, R5.2, R6.2, R7.2, R8.2, R9.2; no longer IC3.AVCC
- net GND: now also ANALONG.4, C2.1, R5.1, R7.1, R8.1, S2.P, S2.P1, S3.P, S3.P1, SEND.3
- net IN: no longer IC3.(INT1)PD3, JP2.5, L298N.5
Other:
- moved on the sheet: JP1, JP2
