File: eagle/7.x/CONTROL PROJECT.sch (EAGLE design)
At the start: 27 parts, among them IC1 MEGA32-P

Commit message: backup
Parts:
- MPU6050: device pinhead:PINHD-1X8 -> pinhead@1:PINHD-1X8
Changed lines of the file:
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@@
 <?xml version="1.0" encoding="utf-8"?>
 <!DOCTYPE eagle SYSTEM "eagle.dtd">
-<eagle version="9.6.2">
+<eagle version="7.7.0">
 <drawing>
 <settings>
 <setting alwaysvectorfont="no"/>
-<setting keepoldvectorfont="yes"/>
 <setting verticaltext="up"/>
 </settings>
@@
 <part name="P+13" library="supply1" deviceset="VCC" device=""/>
 <part name="GND20" library="supply1" deviceset="GND" device=""/>
-<part name="MPU6050" library="pinhead" library_urn="urn:adsk.eagle:library:325" deviceset="PINHD-1X8" device="" package3d_urn="urn:adsk.eagle:package:22409/2"/>
+<part name="MPU6050" library="pinhead@1" deviceset="PINHD-1X8" device=""/>
 </parts>
 <sheets>
@@
 </schematic>
 </drawing>
-<compatibility>
-<note version="8.2" severity="warning">
-Since Version 8.2, EAGLE supports online libraries. The ids
-of those online libraries will not be understood (or retained)
-with this version.
-</note>
-<note version="8.3" severity="warning">
-Since Version 8.3, EAGLE supports URNs for individual library
-assets (packages, symbols, and devices). The URNs of those assets
-will not be understood (or retained) with this version.
-</note>
-<note version="8.3" severity="warning">
-Since Version 8.3, EAGLE supports the association of 3D packages
-with devices in libraries, schematics, and board files. Those 3D
-packages will not be understood (or retained) with this version.
-</note>
-</compatibility>
 </eagle>

Commit message: v7
Connections:
- net N$1 renamed SCL
- net N$13 renamed SDA
- net N$18 renamed SCK
Changed lines of the file:
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@@
 </segment>
 </net>
-<net name="N$1" class="0">
+<net name="SCL" class="0">
 <segment>
 <pinref part="IC1" gate="G$1" pin="(SCL)PC0"/>
@@
 </segment>
 </net>
-<net name="N$13" class="0">
+<net name="SDA" class="0">
 <segment>
 <pinref part="IC1" gate="G$1" pin="(SDA)PC1"/>
@@
 </segment>
 </net>
-<net name="N$18" class="0">
+<net name="SCK" class="0">
 <segment>
 <pinref part="IC1" gate="G$1" pin="(SCK)PB7"/>
@@
 <pinref part="IC1" gate="G$1" pin="(AIN1/OC0)PB3"/>
 <pinref part="L298N" gate="A" pin="1"/>
-<wire x1="-33.02" y1="55.88" x2="-5.08" y2="48.26" width="0.1524" layer="91"/>
-<wire x1="-5.08" y1="48.26" x2="-5.08" y2="-7.62" width="0.1524" layer="91"/>
+<wire x1="-33.02" y1="55.88" x2="-7.62" y2="55.88" width="0.1524" layer="91"/>
+<wire x1="-7.62" y1="55.88" x2="-5.08" y2="-7.62" width="0.1524" layer="91"/>
 </segment>
 </net>
